File: ESP32-BOARD/ESP32-BOARD.kicad_pcb (KiCad board)
At the start: 4 copper layers, 149.9 x 99.8 mm, 148 parts, among them J1 Screw_Terminal_01x08, J2 Input_01x02, J3 Screw_Terminal_01x08, J4 Screw_Terminal_01x08, J5 Conn_01x07_Male, J6 Screw_Terminal_01x04, J7 Screw_Terminal_01x08, J8 DHT11, K1 G5NB-1A-E, K2 G5NB-1A-E, K3 G5NB-1A-E, K4 G5NB-1A-E, K5 G5NB-1A-E, K6 G5NB-1A-E, Q1 MMBT5551, Q2 MMBT5551, Q3 MMBT5551, Q4 MMBT5551, Q5 MMBT5551, Q6 MMBT5551, U1 LM358, U2 LM358, U3 LM2596S-ADJ, U4 LM2596S-ADJ, U5 TLP290-4, U6 TLP290-4, U7 SIM800L, U8 ESP32-dev-board

Commit message: update gerbers and production files
Parts:
- L2, L3, L4, L5, L6, L7: value 15uH -> 10uH
- renumbered K6 to K1, K5 to K2, K4 to K3, K3 to K4, K2 to K5, K1 to K6
Connections:
- C27 pad 1: 4.1V -> /SIM800_PWR
- J8 pad 1: GND -> +3V3
- J8 pad 2: Net-(J8-Pad2) -> /DHT11
- J8 pad 3: /DHT11 -> Net-(J8-Pad3)
- J8 pad 4: +3V3 -> GND
- K3 pad 2: Net-(J7-Pad4) -> /SIM800_PWR
- K3 pad 3: Net-(J7-Pad3) -> 4.1V
- U7 pad 11: 4.1V -> /SIM800_PWR
Routing:
- net /SIM800_PWR: track 0.00 -> 123.4 mm, vias 0 -> 2
- net 4.1V: track 107.4 -> 73.7 mm, vias 4 -> 2
- net Net-(J7-Pad4): track 21.0 -> 0.25 mm
- net Net-(J7-Pad3): track 13.9 -> 0.00 mm
- net GND: track 497.7 -> 504.6 mm
- net +3V3: track 186.2 -> 191.8 mm
- net +5V: track 277.5 -> 272.1 mm
- net /ED_8: track 124.7 -> 126.2 mm
- net /DHT11: track 54.9 -> 53.8 mm
- net /ED_4: track 113.7 -> 113.1 mm
