File: ESP32-BOARD/ESP32-BOARD.sch (KiCad schematic (older format))
At the start: 158 parts, among them J101 Screw_Terminal_01x08, J102 Input_01x02, J103 Screw_Terminal_01x08, J104 Screw_Terminal_01x08, J105 Screw_Terminal_01x04, J106 Screw_Terminal_01x08, J107 Conn_01x07_Male, Q101 BT136-600, Q102 BT136-600, Q103 BT136-600, Q104 BT136-600, U101 LM358, U102 LM358, U103 LM2596S-ADJ, U104 LM2596S-ADJ, U105 TLP290-4, U106 TLP290-4, U107 KAQY214S, U108 KAQY214S, U109 MOC3023S, U110 MOC3023S, U111 MOC3023S, U112 MOC3023S, U113 SIM800L, U114 ESP32-dev-board

Commit message: update on project
Parts:
- removed C101: 1uF, Capacitor_SMD:C_0805_2012Metric, symbol Device:C
- removed C102, C119, C120, C133, C134, C135, C136: 10nF, Capacitor_SMD:C_0805_2012Metric, symbol Device:C
- removed C103, C104, C107, C108, C117, C118: 220uF, Capacitor_SMD:CP_Elec_8x10, symbol Device:CP
- removed C105, C106, C109, C110, C111, C112, C113, C114, C115, C116, C121, C122, C123, C124, C125, C126, C127, C128, C129, C130, C131, C132, C138, C139, C140: 100nF, Capacitor_SMD:C_0805_2012Metric, symbol Device:C
- removed C137: 10uF, Capacitor_SMD:C_0805_2012Metric, symbol Device:C
- removed D101, D102, D103: SS54HF, e-Power:DO-214AC, symbol e-Power:D_SCH_SS54HF
- removed D104, D105, D106, D107, D108, D109: LED, LED_SMD:LED_0805_2012Metric, symbol Device:LED
- removed F101: Fuse, e-Power:FUSE_1206_3216Metric, symbol Device:Fuse
- removed H101, H102, H103, H104: MountingHole_Pad, e-Power:MountingHole_4mm_Pad_Via, symbol Mechanical:MountingHole_Pad
- removed H105: MountingHole_Pad, e-Power:MountingHole_3.2mm_M3_Pad, symbol Mechanical:MountingHole_Pad
- removed J101, J103, J104, J106: Screw_Terminal_01x08, e-Power:TerminalBlock_Phoenix_MKDS-1,5-8-5.08_1x08_P5.08mm_Horizontal, symbol Connector:Screw_Terminal_01x08
- removed J102: Input_01x02, e-Power:TerminalBlock_Phoenix_MKDS-1,5-2_1x02_P5.00mm_Horizontal, symbol Connector:Screw_Terminal_01x02
- removed J105: Screw_Terminal_01x04, e-Power:TerminalBlock_Phoenix_MKDS-1,5-4-5.08_1x04_P5.08mm_Horizontal, symbol Connector:Screw_Terminal_01x04
- removed J107: Conn_01x07_Male, Connector_PinHeader_2.54mm:PinHeader_1x07_P2.54mm_Horizontal, symbol Connector:Conn_01x07_Male
- removed L101: Ferrite, e-Power:FB_0603_1608Metric, symbol Device:L_Core_Ferrite
- removed L102, L103, L104, L105, L106, L107: 15uH, e-Power:L_10.4x10.4_H4.8, symbol e-Power:INDUCTOR_PWR
- removed Q101, Q102, Q103, Q104: BT136-600, Package_TO_SOT_SMD:TO-252-2, symbol Triac_Thyristor:BT136-600
- removed R101, R102, R103, R104: 15R, Resistor_SMD:R_0805_2012Metric, symbol Device:R
- removed R105, R106, R107, R108, R109, R110, R111, R112: 1K, Resistor_SMD:R_0805_2012Metric, symbol Device:R
- removed R113: 2.2R, Resistor_SMD:R_0805_2012Metric, symbol Device:R
- removed R114, R115, R116, R117, R118, R119, R120, R121, R122, R123, R124, R125, R126, R127, R128, R129, R139, R140, R141, R142, R143, R144, R145, R146: 10K, Resistor_SMD:R_0805_2012Metric, symbol Device:R
- removed R130, R132, R135, R136: ADJ, Resistor_SMD:R_0805_2012Metric, symbol Device:R
- removed R131: 1K2, Resistor_SMD:R_0805_2012Metric, symbol Device:R
- removed R133: 3K9, Resistor_SMD:R_0805_2012Metric, symbol Device:R
- removed R134, R153, R154, R155, R156, R157, R158: 100R, Resistor_SMD:R_0805_2012Metric, symbol Device:R
- removed R137: 12K, Resistor_SMD:R_0805_2012Metric, symbol Device:R
- removed R138: 2K7, Resistor_SMD:R_0805_2012Metric, symbol Device:R
- removed R147, R148, R149, R150, R151, R152, R159, R160, R161, R162: 330R, Resistor_SMD:R_0805_2012Metric, symbol Device:R
- removed R163, R164, R165, R166: 470R, Resistor_SMD:R_0805_2012Metric, symbol Device:R
- removed R167, R168, R169, R170: 39R, Resistor_SMD:R_0805_2012Metric, symbol Device:R
- removed R171: 0R, Resistor_SMD:R_0805_2012Metric, symbol Device:R
- removed U101, U102: LM358, Package_SO:SOIC-8_3.9x4.9mm_P1.27mm, symbol Amplifier_Operational:LM358
- removed U103, U104: LM2596S-ADJ, Package_TO_SOT_SMD:TO-263-5_TabPin3, symbol Regulator_Switching:LM2596S-ADJ
- removed U105, U106: TLP290-4, e-Power:SOIC-16_4.55x10.3mm_P1.27mm(TLP290-4), symbol Isolator:TLP290-4
- removed U107, U108: KAQY214S, Package_SO:SO-4_4.4x4.3mm_P2.54mm, symbol Relay_SolidState:ASSR-1218
- removed U109, U110, U111, U112: MOC3023S, Package_DIP:DIP-6_W8.89mm_SMDSocket_LongPads, symbol Relay_SolidState:MOC3023M
- removed U113: SIM800L, e-Power:SIM800L, symbol e-Power:SIM800L
- removed U114: ESP32-dev-board, e-Power:ESP-32-dev-kit, symbol e-Power:ESP32-dev-board
Connections:
- no-connect marks 15 -> 0
Other:
- note removed: "0.0~~3.0V OUTPUTS\n\n"
- note removed: "0.0~~3.3V OUTPUTS\n\n"
- note removed: "0~~24V DIGITAL INPUTS\n"
- note removed: "4~~20mA ANALOG INPUTS\n"
- note removed: "7~~25V"
- note removed: "DIGITAL OUTPUTS\n"
- note removed: "IN: 7~~25V\n"
- note removed: "INPUT\n"
- note removed: "OUT1: 5.0V\n\n"
- note removed: "OUT2: 4.1V\n\n"
- note removed: "VOLTAGE REGULATORS"
- note removed: "gain: 10\n\n\n"

Commit message: modificacoes na placa
Parts:
- added C1: 1uF, Capacitor_SMD:C_0805_2012Metric, symbol Device:C
- added C10, C11, C12, C13, C14, C15, C16, C22, C23, C24, C25, C26, C27, C28, C5, C6, C9: 100nF, Capacitor_SMD:C_0805_2012Metric, symbol Device:C
- added C17, C18, C3, C4, C7, C8: 220uF, Capacitor_SMD:CP_Elec_8x10, symbol Device:CP
- added C19, C2, C20: 10nF, Capacitor_SMD:C_0805_2012Metric, symbol Device:C
- added C21: 10uF, Capacitor_SMD:C_0805_2012Metric, symbol Device:C
- added D1, D10, D11, D12, D13, D14, D15, D2, D3: SS54HF, e-Power:DO-214AC, symbol e-Power:D_SCH_SS54HF
- added D4, D5, D6, D7, D8, D9: LED, LED_SMD:LED_0805_2012Metric, symbol Device:LED
- added F1, F2, F3, F4, F5: Fuse, e-Power:FUSE_1206_3216Metric, symbol Device:Fuse
- added H1, H2, H3, H4: MountingHole_Pad, e-Power:MountingHole_4mm_Pad_Via, symbol Mechanical:MountingHole_Pad
- added H5: MountingHole_Pad, e-Power:MountingHole_3.2mm_M3_Pad, symbol Mechanical:MountingHole_Pad
- added J1, J3, J4, J7: Screw_Terminal_01x08, e-Power:TerminalBlock_Phoenix_MKDS-1,5-8-5.08_1x08_P5.08mm_Horizontal, symbol Connector:Screw_Terminal_01x08
- added J2: Input_01x02, e-Power:TerminalBlock_Phoenix_MKDS-1,5-2_1x02_P5.00mm_Horizontal, symbol Connector:Screw_Terminal_01x02
- added J5: Conn_01x07_Male, Connector_PinHeader_2.54mm:PinHeader_1x07_P2.54mm_Horizontal, symbol Connector:Conn_01x07_Male
- added J6: Screw_Terminal_01x04, e-Power:TerminalBlock_Phoenix_MKDS-1,5-4-5.08_1x04_P5.08mm_Horizontal, symbol Connector:Screw_Terminal_01x04
- added J8: DHT11, Connector_PinHeader_2.54mm:PinHeader_1x04_P2.54mm_Vertical, symbol Connector:Conn_01x04_Male
- added K1, K2, K3, K4, K5, K6: G5NB-1A-E, e-Power:Relay_SPST_Omron-G5Q-1A, symbol e-Power:G5NB-1A-E
- added L1: Ferrite, e-Power:FB_0603_1608Metric, symbol Device:L_Core_Ferrite
- added L2, L3, L4, L5, L6, L7: 15uH, e-Power:L_10.4x10.4_H4.8, symbol e-Power:INDUCTOR_PWR
- added Q1, Q2, Q3, Q4, Q5, Q6: MMBT5551, Package_TO_SOT_SMD:SOT-23, symbol Transistor_BJT:MMBT5551L
- added R1, R2, R3, R4: 15R, Resistor_SMD:R_0805_2012Metric, symbol Device:R
- added R10, R11, R12, R5, R54, R55, R56, R57, R58, R59, R6, R60, R7, R8, R9: 1K, Resistor_SMD:R_0805_2012Metric, symbol Device:R
- added R13: 2.2R, Resistor_SMD:R_0805_2012Metric, symbol Device:R
- added R14, R15, R16, R17, R18, R19, R20, R21, R22, R23, R24, R25, R26, R27, R28, R29, R39, R40, R41, R42, R43, R44, R45, R46: 10K, Resistor_SMD:R_0805_2012Metric, symbol Device:R
- added R30, R32, R35, R36: ADJ, Resistor_SMD:R_0805_2012Metric, symbol Device:R
- added R31: 1K2, Resistor_SMD:R_0805_2012Metric, symbol Device:R
- added R33: 3K9, Resistor_SMD:R_0805_2012Metric, symbol Device:R
- added R34: 100R, Resistor_SMD:R_0805_2012Metric, symbol Device:R
- added R37: 12K, Resistor_SMD:R_0805_2012Metric, symbol Device:R
- added R38: 2K7, Resistor_SMD:R_0805_2012Metric, symbol Device:R
- added R47: 0R, Resistor_SMD:R_0805_2012Metric, symbol Device:R
- added R48, R49, R50, R51, R52, R53: 330R, Resistor_SMD:R_0805_2012Metric, symbol Device:R
- added U1, U2: LM358, Package_SO:SOIC-8_3.9x4.9mm_P1.27mm, symbol Amplifier_Operational:LM358
- added U3, U4: LM2596S-ADJ, Package_TO_SOT_SMD:TO-263-5_TabPin3, symbol Regulator_Switching:LM2596S-ADJ
- added U5, U6: TLP290-4, e-Power:SOIC-16_4.55x10.3mm_P1.27mm(TLP290-4), symbol Isolator:TLP290-4
- added U7: SIM800L, e-Power:SIM800L, symbol e-Power:SIM800L
- added U8: ESP32-dev-board, e-Power:ESP-32-dev-kit, symbol e-Power:ESP32-dev-board
Connections:
- new net: F3.1, J2.1 (Pin_1)
- new net: D1.2 (A), J2.2 (Pin_2)
- new net: D1.1 (K), L1.1
- new net: C2.1, L1.2, L2.1, L3.1, R13.2
- new net: C1.1, R13.1
- new net: C3.1, L3.2, U3.1 (VIN)
- new net: D2.1 (K), L4.1, U3.2 (OUT)
- new net: C6.2, R32.1, R33.1, R36.2, R37.2, U3.4 (FB)
- new net: D3.1 (K), L5.1, U4.2 (OUT)
- new net: C5.2, R30.1, R31.1, R34.2, R35.2, U4.4 (FB)
- new net: C5.1, C8.1, L5.2, L7.1, R35.1, R38.1
- new net: C6.1, C7.1, L4.2, L6.1, R36.1, R37.1
- new net: R34.1, R38.2
- new net: R14.2, R5.1, U1.2 (-)
- new net: R15.1, R6.1, U1.3 (+)
- new net: R17.2, R8.1, U1.5 (+)
- new net: R16.1, R7.1, U1.6 (-)
- new net: J1.8 (Pin_8), R1.2, R6.2
- new net: J1.6 (Pin_6), R2.2, R8.2
- new net: R18.1, R9.1, U2.2 (-)
- new net: R10.1, R19.2, U2.3 (+)
- new net: R12.1, R21.2, U2.5 (+)
- new net: R11.1, R20.1, U2.6 (-)
- new net: J1.4 (Pin_4), R10.2, R3.2
- new net: J1.2 (Pin_2), R12.2, R4.2
- new net: R22.1, U5.1
- new net: R23.1, U5.3
- new net: R24.1, U5.5
- new net: R25.1, U5.7
- new net: J3.7 (Pin_7), R22.2
- new net: J6.1 (Pin_1), K1.3
- new net: J6.2 (Pin_2), K1.2
- new net: J6.3 (Pin_3), K2.3
- new net: J6.4 (Pin_4), K2.2
- new net: D9.2 (A), R53.1
- new net: J3.5 (Pin_5), R23.2
- new net: J3.3 (Pin_3), R24.2
- new net: J3.1 (Pin_1), R25.2
- new net: D8.2 (A), R52.1
- new net: R26.1, U6.1
- new net: R27.1, U6.3
- new net: R29.1, U6.7
- new net: J4.7 (Pin_7), R26.2
- new net: J4.5 (Pin_5), R27.2
- new net: R28.1, U6.5
- new net: J4.3 (Pin_3), R28.2
- new net: J4.1 (Pin_1), R29.2
- new net: D7.2 (A), R51.1
- new net: D6.2 (A), R50.1
- new net: C21.2, U8.2 (ENABLE)
- new net: J7.1 (Pin_1), K3.3
- new net: J7.2 (Pin_2), K3.2
- new net: J7.3 (Pin_3), K4.3
- new net: J7.4 (Pin_4), K4.2
- new net: J7.5 (Pin_5), K5.3
- new net: J7.6 (Pin_6), K5.2
- new net: J7.7 (Pin_7), K6.3
- new net: J7.8 (Pin_8), K6.2
- new net: F1.1, F2.1
- new net: F2.2, F4.2
- new net: F4.1, F5.1
- new net: D15.2 (A), K6.1, Q6.3 (C)
- new net: Q6.1 (B), R59.1
- new net: Q5.1 (B), R58.1
- new net: D14.2 (A), K5.1, Q5.3 (C)
- new net: D13.2 (A), K4.1, Q4.3 (C)
- new net: Q4.1 (B), R57.1
- new net: Q3.1 (B), R56.1
- new net: D12.2 (A), K3.1, Q3.3 (C)
- new net: D5.2 (A), R49.1
- new net: D4.2 (A), R48.1
- new net: D11.2 (A), K2.1, Q2.3 (C)
- new net: Q2.1 (B), R55.1
- new net: Q1.1 (B), R54.1
- new net: D10.2 (A), K1.1, Q1.3 (C)
- new net +3V3: J5.7 (Pin_7), J8.1 (Pin_1), R60.2, U5.10, U5.12, U5.14, U5.16, U6.10, U6.12, U6.14, U6.16, U8.1 (+3V3)
- new net +5V: C17.1, C19.1, C23.1, C25.1, C28.1, D10.1 (K), D11.1 (K), D12.1 (K), D13.1 (K), D14.1 (K), D15.1 (K), K1.5, K2.5, K3.5, K4.5, K5.5, K6.5, L6.2, R47.1, U1.8 (V+), U2.8 (V+)
- new net 4.1V: C18.1, C20.1, C24.1, C27.1, L7.2, U7.11 (VCC)
- new net 5V_u: C22.2, C26.1, J5.5 (Pin_5), R47.2, U8.19 (+5.0V)
- new net CURR_01: R14.1, U1.1, U8.3 (GPIO_36)
- new net CURR_02: R16.2, U1.7, U8.4 (GPIO_39)
- new net CURR_03: R18.2, U2.1, U8.5 (GPIO_34)
- new net CURR_04: R20.2, U2.7, U8.6 (GPIO_35)
- new net DHT11: J8.2 (Pin_2), R60.1, U8.34 (GPIO_3)
- new net ED_1: C9.2, R39.2, U5.15, U8.30 (GPIO_18)
- new net ED_2: C10.2, R40.2, U5.13, U8.29 (GPIO_5)
- new net ED_3: C11.2, R41.2, U5.11, U8.28 (GPIO_17)
- new net ED_4: C12.2, R42.2, U5.9, U8.27 (GPIO_16)
- new net ED_5: C13.2, R43.2, U6.15, U8.23 (GPIO_15)
- new net ED_6: C14.2, R44.2, U6.13, U8.9 (GPIO_25)
- new net ED_7: C15.2, R45.2, U6.11, U8.10 (GPIO_26)
- new net ED_8: C16.2, R46.2, U6.9, U8.11 (GPIO_27)
- new net GND: C1.2, C10.1, C11.1, C12.1, C13.1, C14.1, C15.1, C16.1, C17.2, C18.2, C19.2, C2.2, C20.2, C21.1, C22.1, C23.2, C24.2, C25.2, C26.2, C27.2, C28.2, C3.2, C4.2, C7.2, C8.2, C9.1, D2.2 (A), D3.2 (A), D4.1 (K), D5.1 (K), D6.1 (K), D7.1 (K), D8.1 (K), D9.1 (K), F1.2, F3.2, F5.2, H1.1, H2.1, H3.1, H4.1, H5.1, J1.1 (Pin_1), J1.3 (Pin_3), J1.5 (Pin_5), J1.7 (Pin_7), J5.6 (Pin_6), J8.4 (Pin_4), Q1.2 (E), Q2.2 (E), Q3.2 (E), Q4.2 (E), Q5.2 (E), Q6.2 (E), R1.1, R11.2, R15.2, R17.1, R19.1, R2.1, R21.1, R3.1, R30.2, R31.2, R32.2, R33.2, R39.1, R4.1, R40.1, R41.1, R42.1, R43.1, R44.1, R45.1, R46.1, R5.2, R7.2, R9.2, U1.4 (V-), U2.4 (V-), U3.3 (GND), U3.5 (~ON~/OFF), U4.3 (GND), U4.5 (~ON~/OFF), U5.2, U5.4, U5.6, U5.8, U6.2, U6.4, U6.6, U6.8, U7.7 (GND), U8.32 (GND), U8.38 (GND)
- new net GPIO_12: J5.2 (Pin_2), U8.13 (GPIO_12)
- new net GPIO_14: J5.1 (Pin_1), U8.12 (GPIO_14)
- new net OUT_1: R48.2, R54.2, U8.37 (GPIO_23)
- new net OUT_2: R49.2, R55.2, U8.36 (GPIO_22)
- new net OUT_3: R50.2, R56.2, U8.33 (GPIO_21)
- new net OUT_4: R51.2, R57.2, U8.31 (GPIO_19)
- new net OUT_5: R52.2, R58.2, U8.7 (GPIO_32)
- new net OUT_6: R53.2, R59.2, U8.8 (GPIO_33)
- new net RST_SIM800L: U7.10 (RST), U8.15 (GPIO_13)
- new net RX_SIM800L: U7.9 (RXT), U8.24 (GPIO_2)
- new net SCL: J5.3 (Pin_3), U8.20 (GPIO_6)
- new net SDA: J5.4 (Pin_4), U8.21 (GPIO_7)
- new net TX_SIM800L: U7.8 (TXD), U8.26 (GPIO_4)
- new net VCC: C4.1, J3.2 (Pin_2), J3.4 (Pin_4), J3.6 (Pin_6), J3.8 (Pin_8), J4.2 (Pin_2), J4.4 (Pin_4), J4.6 (Pin_6), J4.8 (Pin_8), L2.2, U4.1 (VIN)
- no-connect marks 0 -> 15
Other:
- note added: "0.0~~3.0V OUTPUTS\n\n"
- note added: "0.0~~3.3V OUTPUTS\n\n"
- note added: "0~~24V DIGITAL INPUTS\n"
- note added: "4~~20mA ANALOG INPUTS\n"
- note added: "7~~25V"
- note added: "IN: 7~~25V\n"
- note added: "INPUT\n"
- note added: "OUT1: 5.0V\n\n"
- note added: "OUT2: 4.1V\n\n"
- note added: "POWER DIGITAL OUTPUTS\n"
- note added: "SPARE FUSES\nFUSÍVEIS RESERVA"
- note added: "VOLTAGE REGULATORS"
- note added: "gain: 10\n\n\n"

Commit message: update gerbers and production files
Parts:
- D4, D5, D6, D7, D8, D9: LCSC C205444 -> C84256
- L2, L3, L4, L5, L6, L7: value 15uH -> 10uH; LCSC C151872 -> C9935
- renumbered K6 to K1, K5 to K2, K4 to K3, K3 to K4, K2 to K5, K1 to K6
Connections:
- net 4.1V: now also K3.3; no longer C27.1, U7.11 (VCC)
- net at J7.3 (Pin_3): no longer K3.3
- net at J7.4 (Pin_4): no longer K3.2
- new net SIM800_PWR: C27.1, K3.2, U7.11 (VCC)
- no-connect marks 15 -> 17
Changed lines of the file:
@@
 P 3450 7800
 F 0 "L3" H 3450 8015 50  0000 C CNN
-F 1 "15uH" H 3450 7924 50  0000 C CNN
+F 1 "10uH" H 3450 7924 50  0000 C CNN
 F 2 "e-Power:L_10.4x10.4_H4.8" H 3450 7675 50  0001 C CNN
-F 3 "https://datasheet.lcsc.com/szlcsc/Sunlord-MWSA1004-330MT_C143966.pdf" H 3450 7800 50  0001 C CNN
-F 4 "C151872" H 3450 7800 50  0001 C CNN "LCSC"
+F 3 "https://datasheet.lcsc.com/szlcsc/1811151526_SXN-Shun-Xiang-Nuo-Elec-SMDRH104R-100MT_C9935.pdf" H 3450 7800 50  0001 C CNN
+F 4 "C9935" H 3450 7800 50  0001 C CNN "LCSC"
 	1    3450 7800
 	1    0    0    -1
@@
 P 6000 9500
 F 0 "L5" H 6000 9600 50  0000 C CNN
-F 1 "15uH" H 6000 9450 50  0000 C CNN
+F 1 "10uH" H 6000 9450 50  0000 C CNN
 F 2 "e-Power:L_10.4x10.4_H4.8" H 6000 9375 50  0001 C CNN
-F 3 "https://datasheet.lcsc.com/szlcsc/Sunlord-MWSA1004-330MT_C143966.pdf" H 6000 9500 50  0001 C CNN
-F 4 "C151872" H 6000 9500 50  0001 C CNN "LCSC"
+F 3 "https://datasheet.lcsc.com/szlcsc/1811151526_SXN-Shun-Xiang-Nuo-Elec-SMDRH104R-100MT_C9935.pdf" H 6000 9500 50  0001 C CNN
+F 4 "C9935" H 6000 9500 50  0001 C CNN "LCSC"
 	1    6000 9500
 	1    0    0    -1
@@
 P 6000 8000
 F 0 "L4" H 6000 8100 50  0000 C CNN
-F 1 "15uH" H 6000 7950 50  0000 C CNN
+F 1 "10uH" H 6000 7950 50  0000 C CNN
 F 2 "e-Power:L_10.4x10.4_H4.8" H 6000 7875 50  0001 C CNN
-F 3 "https://datasheet.lcsc.com/szlcsc/Sunlord-MWSA1004-330MT_C143966.pdf" H 6000 8000 50  0001 C CNN
-F 4 "C151872" H 6000 8000 50  0001 C CNN "LCSC"
+F 3 "https://datasheet.lcsc.com/szlcsc/1811151526_SXN-Shun-Xiang-Nuo-Elec-SMDRH104R-100MT_C9935.pdf" H 6000 8000 50  0001 C CNN
+F 4 "C9935" H 6000 8000 50  0001 C CNN "LCSC"
 	1    6000 8000
 	1    0    0    -1
@@
 P 7000 9500
 F 0 "L7" H 7000 9600 50  0000 C CNN
-F 1 "15uH" H 7000 9450 50  0000 C CNN
+F 1 "10uH" H 7000 9450 50  0000 C CNN
 F 2 "e-Power:L_10.4x10.4_H4.8" H 7000 9375 50  0001 C CNN
-F 3 "https://datasheet.lcsc.com/szlcsc/Sunlord-MWSA1004-330MT_C143966.pdf" H 7000 9500 50  0001 C CNN
-F 4 "C151872" H 7000 9500 50  0001 C CNN "LCSC"
+F 3 "https://datasheet.lcsc.com/szlcsc/1811151526_SXN-Shun-Xiang-Nuo-Elec-SMDRH104R-100MT_C9935.pdf" H 7000 9500 50  0001 C CNN
+F 4 "C9935" H 7000 9500 50  0001 C CNN "LCSC"
 	1    7000 9500
 	1    0    0    -1
@@
 P 7000 8000
 F 0 "L6" H 7000 8100 50  0000 C CNN
-F 1 "15uH" H 7000 7950 50  0000 C CNN
+F 1 "10uH" H 7000 7950 50  0000 C CNN
 F 2 "e-Power:L_10.4x10.4_H4.8" H 7000 7875 50  0001 C CNN
-F 3 "https://datasheet.lcsc.com/szlcsc/Sunlord-MWSA1004-330MT_C143966.pdf" H 7000 8000 50  0001 C CNN
-F 4 "C151872" H 7000 8000 50  0001 C CNN "LCSC"
+F 3 "https://datasheet.lcsc.com/szlcsc/1811151526_SXN-Shun-Xiang-Nuo-Elec-SMDRH104R-100MT_C9935.pdf" H 7000 8000 50  0001 C CNN
+F 4 "C9935" H 7000 8000 50  0001 C CNN "LCSC"
 	1    7000 8000
 	1    0    0    -1
@@
 Text Label 9900 5950 0    50   ~ 0
 TX_SIM800L
-Text GLabel 9900 5350 1    50   Input ~ 0
+Text GLabel 14100 6450 2    50   Input ~ 0
 4.1V
 $Comp
@@
 	10000 5450 9900 5450
 Connection ~ 9900 5450
-Wire Wire Line
-	9900 5450 9900 5350
 $Comp
 L power:GND #PWR077
@@
 F 1 "LED" V 12000 5900 50  0000 R CNN
 F 2 "LED_SMD:LED_0805_2012Metric" H 11950 5950 50  0001 C CNN
-F 3 "https://datasheet.lcsc.com/szlcsc/1811011120_Orient-ORH-R35A_C205444.pdf" H 11950 5950 50  0001 C CNN
-F 4 "C205444" V 11950 5950 50  0001 C CNN "LCSC"
+F 3 "" H 11950 5950 50  0001 C CNN
+F 4 "C84256" V 11950 5950 50  0001 C CNN "LCSC"
 F 5 "" V 11950 5950 50  0001 C CNN "Field5"
 	1    11950 5950
@@
 F 1 "LED" V 12000 6950 50  0000 R CNN
 F 2 "LED_SMD:LED_0805_2012Metric" H 11950 7000 50  0001 C CNN
-F 3 "https://datasheet.lcsc.com/szlcsc/1811011120_Orient-ORH-R35A_C205444.pdf" H 11950 7000 50  0001 C CNN
-F 4 "C205444" V 11950 7000 50  0001 C CNN "LCSC"
+F 3 "" H 11950 7000 50  0001 C CNN
+F 4 "C84256" V 11950 7000 50  0001 C CNN "LCSC"
 F 5 "" V 11950 7000 50  0001 C CNN "Field5"
 	1    11950 7000
@@
 F 1 "LED" V 12000 8000 50  0000 R CNN
 F 2 "LED_SMD:LED_0805_2012Metric" H 11950 8050 50  0001 C CNN
-F 3 "https://datasheet.lcsc.com/szlcsc/1811011120_Orient-ORH-R35A_C205444.pdf" H 11950 8050 50  0001 C CNN
-F 4 "C205444" V 11950 8050 50  0001 C CNN "LCSC"
+F 3 "" H 11950 8050 50  0001 C CNN
+F 4 "C84256" V 11950 8050 50  0001 C CNN "LCSC"
 F 5 "" V 11950 8050 50  0001 C CNN "Field5"
 	1    11950 8050
@@
 F 1 "LED" V 12000 9050 50  0000 R CNN
 F 2 "LED_SMD:LED_0805_2012Metric" H 11950 9100 50  0001 C CNN
-F 3 "https://datasheet.lcsc.com/szlcsc/1811011120_Orient-ORH-R35A_C205444.pdf" H 11950 9100 50  0001 C CNN
-F 4 "C205444" V 11950 9100 50  0001 C CNN "LCSC"
+F 3 "" H 11950 9100 50  0001 C CNN
+F 4 "C84256" V 11950 9100 50  0001 C CNN "LCSC"
 F 5 "" V 11950 9100 50  0001 C CNN "Field5"
 	1    11950 9100
@@
 P 3400 9300
 F 0 "L2" H 3400 9515 50  0000 C CNN
-F 1 "15uH" H 3400 9424 50  0000 C CNN
+F 1 "10uH" H 3400 9424 50  0000 C CNN
 F 2 "e-Power:L_10.4x10.4_H4.8" H 3400 9175 50  0001 C CNN
-F 3 "https://datasheet.lcsc.com/szlcsc/Sunlord-MWSA1004-330MT_C143966.pdf" H 3400 9300 50  0001 C CNN
-F 4 "C151872" H 3400 9300 50  0001 C CNN "LCSC"
+F 3 "https://datasheet.lcsc.com/szlcsc/1811151526_SXN-Shun-Xiang-Nuo-Elec-SMDRH104R-100MT_C9935.pdf" H 3400 9300 50  0001 C CNN
+F 4 "C9935" H 3400 9300 50  0001 C CNN "LCSC"
 	1    3400 9300
 	1    0    0    -1
@@
 SPARE FUSES\nFUSÍVEIS RESERVA
 $Comp
-L e-Power:G5NB-1A-E K6
+L e-Power:G5NB-1A-E K1
 U 1 1 60896A22
 P 13800 9000
-F 0 "K6" H 14200 9000 50  0000 L CNN
+F 0 "K1" H 14200 9000 50  0000 L CNN
 F 1 "G5NB-1A-E" V 14150 9000 50  0000 C CNN
 F 2 "e-Power:Relay_SPST_Omron-G5Q-1A" H 14150 8950 50  0001 L CNN
@@
 $EndComp
 $Comp
-L e-Power:G5NB-1A-E K5
+L e-Power:G5NB-1A-E K2
 U 1 1 60C9EF54
 P 13800 7950
-F 0 "K5" H 14200 7950 50  0000 L CNN
+F 0 "K2" H 14200 7950 50  0000 L CNN
 F 1 "G5NB-1A-E" V 14150 7950 50  0000 C CNN
 F 2 "e-Power:Relay_SPST_Omron-G5Q-1A" H 14150 7900 50  0001 L CNN
@@
 $EndComp
 $Comp
-L e-Power:G5NB-1A-E K4
+L e-Power:G5NB-1A-E K3
 U 1 1 60FA2202
 P 13800 6900
-F 0 "K4" H 14200 6900 50  0000 L CNN
+F 0 "K3" H 14200 6900 50  0000 L CNN
 F 1 "G5NB-1A-E" V 14150 6900 50  0000 C CNN
 F 2 "e-Power:Relay_SPST_Omron-G5Q-1A" H 14150 6850 50  0001 L CNN
@@
 $EndComp
 $Comp
-L e-Power:G5NB-1A-E K3
+L e-Power:G5NB-1A-E K4
 U 1 1 60FA227C
 P 13800 5850
-F 0 "K3" H 14200 5850 50  0000 L CNN
+F 0 "K4" H 14200 5850 50  0000 L CNN
 F 1 "G5NB-1A-E" V 14150 5850 50  0000 C CNN
 F 2 "e-Power:Relay_SPST_Omron-G5Q-1A" H 14150 5800 50  0001 L CNN
@@
 F 1 "LED" V 12000 3800 50  0000 R CNN
 F 2 "LED_SMD:LED_0805_2012Metric" H 11950 3850 50  0001 C CNN
-F 3 "https://datasheet.lcsc.com/szlcsc/1811011120_Orient-ORH-R35A_C205444.pdf" H 11950 3850 50  0001 C CNN
-F 4 "C205444" V 11950 3850 50  0001 C CNN "LCSC"
+F 3 "" H 11950 3850 50  0001 C CNN
+F 4 "C84256" V 11950 3850 50  0001 C CNN "LCSC"
 F 5 "" V 11950 3850 50  0001 C CNN "Field5"
 	1    11950 3850
@@
 F 1 "LED" V 12000 4850 50  0000 R CNN
 F 2 "LED_SMD:LED_0805_2012Metric" H 11950 4900 50  0001 C CNN
-F 3 "https://datasheet.lcsc.com/szlcsc/1811011120_Orient-ORH-R35A_C205444.pdf" H 11950 4900 50  0001 C CNN
-F 4 "C205444" V 11950 4900 50  0001 C CNN "LCSC"
+F 3 "" H 11950 4900 50  0001 C CNN
+F 4 "C84256" V 11950 4900 50  0001 C CNN "LCSC"
 F 5 "" V 11950 4900 50  0001 C CNN "Field5"
 	1    11950 4900
@@
 $EndComp
 $Comp
-L e-Power:G5NB-1A-E K2
+L e-Power:G5NB-1A-E K5
 U 1 1 61324F87
 P 13800 4800
-F 0 "K2" H 14200 4800 50  0000 L CNN
+F 0 "K5" H 14200 4800 50  0000 L CNN
 F 1 "G5NB-1A-E" V 14150 4800 50  0000 C CNN
 F 2 "e-Power:Relay_SPST_Omron-G5Q-1A" H 14150 4750 50  0001 L CNN
@@
 $EndComp
 $Comp
-L e-Power:G5NB-1A-E K1
+L e-Power:G5NB-1A-E K6
 U 1 1 61325000
 P 13800 3750
-F 0 "K1" H 14200 3750 50  0000 L CNN
+F 0 "K6" H 14200 3750 50  0000 L CNN
 F 1 "G5NB-1A-E" V 14150 3750 50  0000 C CNN
 F 2 "e-Power:Relay_SPST_Omron-G5Q-1A" H 14150 3700 50  0001 L CNN
@@
 	14000 7450 14950 7450
 Wire Wire Line
-	14000 7200 14000 7350
-Wire Wire Line
-	14000 7350 14950 7350
-Wire Wire Line
-	14950 7250 14450 7250
-Wire Wire Line
-	14450 7250 14450 6550
-Wire Wire Line
-	14450 6550 14000 6550
-Wire Wire Line
-	14000 6550 14000 6600
+	14000 7200 14000 7300
 Wire Wire Line
 	14950 7150 14500 7150
@@
 	10150 1450 10050 1450
 Connection ~ 10050 1450
+NoConn ~ 14950 7350
+NoConn ~ 14950 7250
+Wire Wire Line
+	14100 6450 14000 6450
+Wire Wire Line
+	14000 6450 14000 6600
+Wire Wire Line
+	14000 7300 14100 7300
+Text Label 14100 7300 0    50   ~ 0
+SIM800_PWR
+Text Label 9900 5200 0    50   ~ 0
+SIM800_PWR
+Wire Wire Line
+	9900 5200 9900 5450
 $EndSCHEMATC
